Commit message: missed option for proximity sensors in inail 2 arm without dagana

File: inail2arm_urdf/config/inail2arm.urdf.xacro (robot description, xacro)
@@ -9,3 +9,5 @@
 <!-- In future, xbot will be able to ignore end-effectors in the hal and this should not be neccesary anymore -->
 <xacro:property name="DAGANA_STANDALONE_PLUGIN" value="true" />
+<xacro:arg name="proximity_sensors" default="true"/>
+<xacro:property name="PROXIMITY_SENSORS" value="$(arg proximity_sensors)" />
 </robot>

Commit message: changes for arm without dagana

File: inail2arm_urdf/config/inail2arm.urdf.xacro (robot description, xacro)
@@ -8,5 +8,5 @@
 <!-- This property is used in the gazebo/xbot.gazebo.xacro file -->
 <!-- In future, xbot will be able to ignore end-effectors in the hal and this should not be neccesary anymore -->
-<xacro:property name="DAGANA_STANDALONE_PLUGIN" value="true" />
+<xacro:property name="DAGANA_STANDALONE_PLUGIN" value="false" />
 <xacro:arg name="proximity_sensors" default="true"/>
 <xacro:property name="PROXIMITY_SENSORS" value="$(arg proximity_sensors)" />
