Commit message: dagana color can stay on dagana xacro

File: inail2arm_urdf/urdf/gazebo/materials.gazebo.xacro (robot description, xacro)
@@ -25,11 +25,3 @@
 	</gazebo>
 </xacro:if>
-<xacro:if value="${END_EFFECTOR == 'dagana' or END_EFFECTOR == 'dagana_fixed'}">
-	<gazebo reference="dagana_1_top_link">
-		<material>Gazebo/BlackTransparent</material>
-	</gazebo>
-	<gazebo reference="dagana_1_bottom_link">
-		<material>Gazebo/BlackTransparent</material>
-	</gazebo>
-</xacro:if>
 </robot>
