Commit message: fix mounting dagana

File: inail2arm_urdf/urdf/kinematics_properties.urdf.xacro (robot description, xacro)
@@ -50,5 +50,5 @@
 <xacro:property name="EE_mount_roll" value=" 0.0 "/>
 <xacro:property name="EE_mount_pitch" value=" 0.0 "/>
-<xacro:property name="EE_mount_yaw" value=" 0.0 "/>
+<xacro:property name="EE_mount_yaw" value=" ${PI/2} "/>
 <!-- Origin -->
 <xacro:property name="No_end_ft_Ox" value=" 0.0 "/>
