Commit message: no dashes for isaac

File: inail2arm_urdf/urdf/inail2arm_macro.urdf.xacro (robot description, xacro)
@@ -15,13 +15,13 @@
             <origin xyz="0.0 0.0 0.0" rpy="0.0 0.0 0.0" />
             <geometry>
-               <mesh filename="package://inail2arm_urdf/meshes/mesh_shoulder-yaw.stl"
-                  scale="0.001 ${rot*0.001} 0.001" />
-            </geometry>
-            <material name="blue" />
-         </visual>
-         <collision>
-            <origin xyz="0.0 0.0 0.0" rpy="0.0 0.0 0.0" />
-            <geometry>
-               <mesh filename="package://inail2arm_urdf/meshes/simple/mesh_shoulder-yaw.stl"
+               <mesh filename="package://inail2arm_urdf/meshes/mesh_shoulder_yaw.stl"
+                  scale="0.001 ${rot*0.001} 0.001" />
+            </geometry>
+            <material name="blue" />
+         </visual>
+         <collision>
+            <origin xyz="0.0 0.0 0.0" rpy="0.0 0.0 0.0" />
+            <geometry>
+               <mesh filename="package://inail2arm_urdf/meshes/simple/mesh_shoulder_yaw.stl"
                   scale="0.001 ${rot*0.001} 0.001" />
             </geometry>
@@ -40,13 +40,13 @@
             <origin xyz="0.0 0.0 0.0" rpy="0.0 0.0 0.0" />
             <geometry>
-               <mesh filename="package://inail2arm_urdf/meshes/mesh_shoulder-pitch.stl"
-                  scale="0.001 ${rot*0.001} 0.001" />
-            </geometry>
-            <material name="blue" />
-         </visual>
-         <collision>
-            <origin xyz="0.0 0.0 0.0" rpy="0.0 0.0 0.0" />
-            <geometry>
-               <mesh filename="package://inail2arm_urdf/meshes/simple/mesh_shoulder-pitch.stl"
+               <mesh filename="package://inail2arm_urdf/meshes/mesh_shoulder_pitch.stl"
+                  scale="0.001 ${rot*0.001} 0.001" />
+            </geometry>
+            <material name="blue" />
+         </visual>
+         <collision>
+            <origin xyz="0.0 0.0 0.0" rpy="0.0 0.0 0.0" />
+            <geometry>
+               <mesh filename="package://inail2arm_urdf/meshes/simple/mesh_shoulder_pitch.stl"
                   scale="0.001 ${rot*0.001} 0.001" />
             </geometry>
@@ -90,13 +90,13 @@
             <origin xyz="0.0 0.0 0.0" rpy="0.0 0.0 0.0" />
             <geometry>
-               <mesh filename="package://inail2arm_urdf/meshes/mesh_forearm-yaw.stl"
-                  scale="0.001 ${rot*0.001} 0.001" />
-            </geometry>
-            <material name="blue" />
-         </visual>
-         <collision>
-            <origin xyz="0.0 0.0 0.0" rpy="0.0 0.0 0.0" />
-            <geometry>
-               <mesh filename="package://inail2arm_urdf/meshes/simple/mesh_forearm-yaw.stl"
+               <mesh filename="package://inail2arm_urdf/meshes/mesh_forearm_yaw.stl"
+                  scale="0.001 ${rot*0.001} 0.001" />
+            </geometry>
+            <material name="blue" />
+         </visual>
+         <collision>
+            <origin xyz="0.0 0.0 0.0" rpy="0.0 0.0 0.0" />
+            <geometry>
+               <mesh filename="package://inail2arm_urdf/meshes/simple/mesh_forearm_yaw.stl"
                   scale="0.001 ${rot*0.001} 0.001" />
             </geometry>
@@ -116,5 +116,5 @@
             <geometry>
                <mesh
-                  filename="package://inail2arm_urdf/meshes/mesh_wrist-pitch.stl"
+                  filename="package://inail2arm_urdf/meshes/mesh_wrist_pitch.stl"
                   scale="0.001
                ${rot*0.001} 0.001" />
@@ -126,5 +126,5 @@
             <geometry>
                <mesh
-                  filename="package://inail2arm_urdf/meshes/simple/mesh_wrist-pitch.stl"
+                  filename="package://inail2arm_urdf/meshes/simple/mesh_wrist_pitch.stl"
                   scale="0.001
                ${rot*0.001} 0.001" />
@@ -143,14 +143,14 @@
             <geometry>
                <mesh
-                  filename="package://inail2arm_urdf/meshes/mesh_wrist-roll.stl"
-                  scale="0.001 ${rot*0.001} 0.001" />
-            </geometry>
-            <material name="blue" />
-         </visual>
-         <collision>
-            <origin xyz="0.0 0.0 0.0" rpy="0.0 0.0 0.0" />
-            <geometry>
-               <mesh
-                  filename="package://inail2arm_urdf/meshes/simple/mesh_wrist-roll.stl"
+                  filename="package://inail2arm_urdf/meshes/mesh_wrist_roll.stl"
+                  scale="0.001 ${rot*0.001} 0.001" />
+            </geometry>
+            <material name="blue" />
+         </visual>
+         <collision>
+            <origin xyz="0.0 0.0 0.0" rpy="0.0 0.0 0.0" />
+            <geometry>
+               <mesh
+                  filename="package://inail2arm_urdf/meshes/simple/mesh_wrist_roll.stl"
                   scale="0.001 ${rot*0.001} 0.001" />
             </geometry>
