Commit message: ball better tcp

File: inail2arm_urdf/urdf/ball.urdf.xacro (robot description, xacro)
@@ -31,5 +31,5 @@
 	<parent link="ball${arm_num}"/>
 	<child link="ball${arm_num}_tip"/>
-	<origin xyz="0 0 -0.07" rpy="0 0 0"/>
+	<origin xyz="0 0 -0.078" rpy="0 0 0"/>
 </joint>
 </xacro:macro>

Commit message: inail2arm ros2 version update

File: inail2arm_urdf/urdf/ball.urdf.xacro (robot description, xacro)
@@ -11,5 +11,5 @@
       <origin xyz="0.0 0.0 0.0" rpy="0.0 0.0 0.0"/>
       <geometry name="ball${arm_num}_visual">
-        <mesh filename="package://inail2arm_urdf/meshes/BallHand.stl" scale="0.001 0.001 0.001" />
+        <mesh filename="file://$(find inail2arm_urdf)/meshes/BallHand.stl" scale="0.001 0.001 0.001" />
       </geometry>
       <material name="dark_grey"/>
@@ -18,5 +18,5 @@
       <origin xyz="0.0 0.0 0.0" rpy="0.0 0.0 0.0"/>
       <geometry name="ball${arm_num}_collision">
-        <mesh filename="package://inail2arm_urdf/meshes/simple/BallHand.stl" scale="0.001 0.001 0.001" />
+        <mesh filename="file://$(find inail2arm_urdf)/meshes/simple/BallHand.stl" scale="0.001 0.001 0.001" />
       </geometry>
    </collision>

File: inail2arm_urdf/urdf/gazebo/xbot.gazebo.xacro (robot description, xacro)
@@ -1,21 +1,19 @@
 <?xml version="1.0"?>
 <robot xmlns:xacro="http://ros.org/wiki/xacro">
-<gazebo>
-    <plugin name="xbot2_joint_driver" filename="libxbot2_gz_joint_server.so">
-        <pid>
-            <gain name="lowpwr_mot" p="50"  d="5"/>
-            <gain name="small_mot"  p="600"  d="6"/>
-            <gain name="medium_mot" p="4000" d="40"/>
-            <gain name="big_mot"    p="8000" d="50"/>
-            <gain name="dagana_mot"  p="10" d="0.5"/>
-            <pid name="j_arm1_1" profile="medium_mot"/>
-            <pid name="j_arm1_2" profile="medium_mot"/>
-            <pid name="j_arm1_3" profile="medium_mot"/>
-            <pid name="j_arm1_4" profile="medium_mot"/>
-            <pid name="j_arm1_5" profile="small_mot"/>
-            <pid name="j_arm1_6" profile="small_mot"/>
-            <pid name="dagana_1_claw_joint" profile="dagana_mot"/>
-        </pid>
-    </plugin>
-</gazebo>
+    <gazebo>
+        <plugin filename="xbot2_gz_joint_server" name="gz::sim::systems::GzJointServer">
+                <profile name="lowpwr_mot" p="50"  d="5"/>
+                <profile name="small_mot"  p="600"  d="6"/>
+                <profile name="medium_mot" p="4000" d="40"/>
+                <profile name="big_mot"    p="8000" d="50"/>
+                <profile name="dagana_mot"  p="10" d="0.5"/>
+                <pid name="j_arm1_1" profile="medium_mot"/>
+                <pid name="j_arm1_2" profile="medium_mot"/>
+                <pid name="j_arm1_3" profile="medium_mot"/>
+                <pid name="j_arm1_4" profile="medium_mot"/>
+                <pid name="j_arm1_5" profile="small_mot"/>
+                <pid name="j_arm1_6" profile="small_mot"/>
+                <pid name="dagana_1_claw_joint" profile="dagana_mot"/>
+        </plugin>
+    </gazebo>
 </robot>

File: inail2arm_urdf/urdf/inail2arm_macro.urdf.xacro (robot description, xacro)
@@ -15,13 +15,13 @@
             <origin xyz="0.0 0.0 0.0" rpy="0.0 0.0 0.0" />
             <geometry>
-               <mesh filename="package://inail2arm_urdf/meshes/mesh_shoulder_yaw.stl"
-                  scale="0.001 ${rot*0.001} 0.001" />
-            </geometry>
-            <material name="blue" />
-         </visual>
-         <collision>
-            <origin xyz="0.0 0.0 0.0" rpy="0.0 0.0 0.0" />
-            <geometry>
-               <mesh filename="package://inail2arm_urdf/meshes/simple/mesh_shoulder_yaw.stl"
+               <mesh filename="file://$(find inail2arm_urdf)/meshes/mesh_shoulder_yaw.stl"
+                  scale="0.001 ${rot*0.001} 0.001" />
+            </geometry>
+            <material name="blue" />
+         </visual>
+         <collision>
+            <origin xyz="0.0 0.0 0.0" rpy="0.0 0.0 0.0" />
+            <geometry>
+               <mesh filename="file://$(find inail2arm_urdf)/meshes/simple/mesh_shoulder_yaw.stl"
                   scale="0.001 ${rot*0.001} 0.001" />
             </geometry>
@@ -40,13 +40,13 @@
             <origin xyz="0.0 0.0 0.0" rpy="0.0 0.0 0.0" />
             <geometry>
-               <mesh filename="package://inail2arm_urdf/meshes/mesh_shoulder_pitch.stl"
-                  scale="0.001 ${rot*0.001} 0.001" />
-            </geometry>
-            <material name="blue" />
-         </visual>
-         <collision>
-            <origin xyz="0.0 0.0 0.0" rpy="0.0 0.0 0.0" />
-            <geometry>
-               <mesh filename="package://inail2arm_urdf/meshes/simple/mesh_shoulder_pitch.stl"
+               <mesh filename="file://$(find inail2arm_urdf)/meshes/mesh_shoulder_pitch.stl"
+                  scale="0.001 ${rot*0.001} 0.001" />
+            </geometry>
+            <material name="blue" />
+         </visual>
+         <collision>
+            <origin xyz="0.0 0.0 0.0" rpy="0.0 0.0 0.0" />
+            <geometry>
+               <mesh filename="file://$(find inail2arm_urdf)/meshes/simple/mesh_shoulder_pitch.stl"
                   scale="0.001 ${rot*0.001} 0.001" />
             </geometry>
@@ -65,13 +65,13 @@
             <origin xyz="0.0 0.0 0.0" rpy="0.0 0.0 0.0" />
             <geometry>
-               <mesh filename="package://inail2arm_urdf/meshes/mesh_elbow.stl"
-                  scale="0.001 ${rot*0.001} 0.001" />
-            </geometry>
-            <material name="blue" />
-         </visual>
-         <collision>
-            <origin xyz="0.0 0.0 0.0" rpy="0.0 0.0 0.0" />
-            <geometry>
-               <mesh filename="package://inail2arm_urdf/meshes/simple/mesh_elbow.stl"
+               <mesh filename="file://$(find inail2arm_urdf)/meshes/mesh_elbow.stl"
+                  scale="0.001 ${rot*0.001} 0.001" />
+            </geometry>
+            <material name="blue" />
+         </visual>
+         <collision>
+            <origin xyz="0.0 0.0 0.0" rpy="0.0 0.0 0.0" />
+            <geometry>
+               <mesh filename="file://$(find inail2arm_urdf)/meshes/simple/mesh_elbow.stl"
                   scale="0.001 ${rot*0.001} 0.001" />
             </geometry>
@@ -90,13 +90,13 @@
             <origin xyz="0.0 0.0 0.0" rpy="0.0 0.0 0.0" />
             <geometry>
-               <mesh filename="package://inail2arm_urdf/meshes/mesh_forearm_yaw.stl"
-                  scale="0.001 ${rot*0.001} 0.001" />
-            </geometry>
-            <material name="blue" />
-         </visual>
-         <collision>
-            <origin xyz="0.0 0.0 0.0" rpy="0.0 0.0 0.0" />
-            <geometry>
-               <mesh filename="package://inail2arm_urdf/meshes/simple/mesh_forearm_yaw.stl"
+               <mesh filename="file://$(find inail2arm_urdf)/meshes/mesh_forearm_yaw.stl"
+                  scale="0.001 ${rot*0.001} 0.001" />
+            </geometry>
+            <material name="blue" />
+         </visual>
+         <collision>
+            <origin xyz="0.0 0.0 0.0" rpy="0.0 0.0 0.0" />
+            <geometry>
+               <mesh filename="file://$(find inail2arm_urdf)/meshes/simple/mesh_forearm_yaw.stl"
                   scale="0.001 ${rot*0.001} 0.001" />
             </geometry>
@@ -116,5 +116,5 @@
             <geometry>
                <mesh
-                  filename="package://inail2arm_urdf/meshes/mesh_wrist_pitch.stl"
+                  filename="file://$(find inail2arm_urdf)/meshes/mesh_wrist_pitch.stl"
                   scale="0.001
                ${rot*0.001} 0.001" />
@@ -126,5 +126,5 @@
             <geometry>
                <mesh
-                  filename="package://inail2arm_urdf/meshes/simple/mesh_wrist_pitch.stl"
+                  filename="file://$(find inail2arm_urdf)/meshes/simple/mesh_wrist_pitch.stl"
                   scale="0.001
                ${rot*0.001} 0.001" />
@@ -143,14 +143,14 @@
             <geometry>
                <mesh
-                  filename="package://inail2arm_urdf/meshes/mesh_wrist_roll.stl"
-                  scale="0.001 ${rot*0.001} 0.001" />
-            </geometry>
-            <material name="blue" />
-         </visual>
-         <collision>
-            <origin xyz="0.0 0.0 0.0" rpy="0.0 0.0 0.0" />
-            <geometry>
-               <mesh
-                  filename="package://inail2arm_urdf/meshes/simple/mesh_wrist_roll.stl"
+                  filename="file://$(find inail2arm_urdf)/meshes/mesh_wrist_roll.stl"
+                  scale="0.001 ${rot*0.001} 0.001" />
+            </geometry>
+            <material name="blue" />
+         </visual>
+         <collision>
+            <origin xyz="0.0 0.0 0.0" rpy="0.0 0.0 0.0" />
+            <geometry>
+               <mesh
+                  filename="file://$(find inail2arm_urdf)/meshes/simple/mesh_wrist_roll.stl"
                   scale="0.001 ${rot*0.001} 0.001" />
             </geometry>

File: inail2arm_urdf/urdf/inail2base.urdf.xacro (robot description, xacro)
@@ -13,5 +13,5 @@
                 <origin xyz="0.0 0.0 0.0" rpy="0.0 0.0 0.0" />
                 <geometry>
-                    <mesh filename="package://inail2arm_urdf/meshes/mesh_base.stl"
+                    <mesh filename="file://$(find inail2arm_urdf)/meshes/mesh_base.stl"
                         scale="0.001 ${rot*0.001} 0.001" />
                 </geometry>
@@ -21,5 +21,5 @@
                 <origin xyz="0.0 0.0 0.0" rpy="0.0 0.0 0.0" />
                 <geometry>
-                    <mesh filename="package://inail2arm_urdf/meshes/simple/mesh_base.stl"
+                    <mesh filename="file://$(find inail2arm_urdf)/meshes/simple/mesh_base.stl"
                         scale="0.001 ${rot*0.001} 0.001" />
                 </geometry>
