Commit message: toward mergin into devel

File: inail2arm_srdf/srdf/inail2arm.srdf.xacro (robot description, xacro)
@@ -23,7 +23,4 @@
         <joint name="j_arm1_5" value="1.1"/>
         <joint name="j_arm1_6" value="0.0"/>
-<!--        <xacro:if value="${END_EFFECTOR == 'dagana'}">
-            <joint name="dagana_1_bottom_link" value="0.0"/>
-        </xacro:if>-->
     </group_state>
     <!--  For moveit    -->

File: inail2arm_urdf/config/inail2arm.urdf.xacro (robot description, xacro)
@@ -3,11 +3,7 @@
 <xacro:property name="model_name" value="inail2arm" />
 <xacro:property name="model_version" value="0.1" />
-<xacro:arg name="end_effector" default="dagana"/> <!-- none, ball, dagana_fixed, dagana -->
+<xacro:arg name="end_effector" default="none"/> <!-- none, ball, dagana_fixed, dagana -->
 <xacro:property name="END_EFFECTOR" value="$(arg end_effector)" />
-<!-- HACK to add standalone dagana plugin and ignore the dagana joint in the libxbot2_gz_joint_server -->
-<!-- This property is used in the gazebo/xbot.gazebo.xacro file -->
-<!-- In future, xbot will be able to ignore end-effectors in the hal and this should not be neccesary anymore -->
-<xacro:property name="DAGANA_STANDALONE_PLUGIN" value="false" />
-<xacro:arg name="proximity_sensors" default="true"/>
+<xacro:arg name="proximity_sensors" default="false"/>
 <xacro:property name="PROXIMITY_SENSORS" value="$(arg proximity_sensors)" />
 </robot>

Commit message: nicla option necessary for ignoring collisions

File: inail2arm_srdf/srdf/inail2arm.srdf.xacro (robot description, xacro)
@@ -59,4 +59,8 @@
         <disable_collisions link1="arm1_6" link2="dagana_1_top_link" reason="Adjacent"/>
         <disable_collisions link1="dagana_1_bottom_link" link2="dagana_1_top_link" reason="Adjacent"/>
+        <xacro:if value="${NICLA}">
+            <disable_collisions link1="dagana_1_bottom_link" link2="nicla_base" reason="Adjacent"/>
+            <disable_collisions link1="dagana_1_top_link" link2="nicla_base" reason="Adjacent"/>
+        </xacro:if>
     </xacro:if>
 </robot>

File: inail2arm_urdf/config/inail2arm.urdf.xacro (robot description, xacro)
@@ -5,4 +5,6 @@
 <xacro:arg name="end_effector" default="none"/> <!-- none, ball, dagana_fixed, dagana -->
 <xacro:property name="END_EFFECTOR" value="$(arg end_effector)" />
+<xacro:arg name="nicla" default="false"/> <!-- the nicla inside the dagana-->
+<xacro:property name="NICLA" value="$(arg nicla)" />
 <xacro:arg name="proximity_sensors" default="false"/>
 <xacro:property name="PROXIMITY_SENSORS" value="$(arg proximity_sensors)" />
